Commit message: Add files via upload

File: floating_robotiq_2f_85.urdf (robot description, URDF)
Before this commit: robot robotiq_arg2f_85_model, 17 links, 16 joints
Joints:
- joint left_outer_knuckle_joint: limit lower=0 upper=0.8 effort=1000 velocity=2.0 -> lower=0 upper=0.81 effort=1000 velocity=2.0

File: robotiq_2f_85.urdf (robot description, URDF)
Before this commit: robot robotiq_arg2f_85_model, 11 links, 10 joints
Joints:
- joint left_outer_knuckle_joint: limit lower=0 upper=0.8 effort=1000 velocity=2.0 -> lower=0 upper=0.81 effort=1000 velocity=2.0
